File: hardware/logic-analyzer.kicad_sch (KiCad schematic)
At the start: 100 parts, among them J1 USB_C_Receptacle, J2 Conn_02x20, J3 Conn_02x04, J4 Conn_02x15, J5 Conn_02x15, SW1 SW_Push, SW2 SW_Push, U1 CH32H417MxUx, U16 TPD4EUSB30, U2 AMS1117-3.3, U22 TPD4EUSB30, U23 TPD4EUSB30, U3 LMV321, U5 TMUXHS4212, Y1 25MHz 20pF

Commit message: Stash
Parts:
- H1, H2: now not fitted
- J2, J3, J4, J5: now not fitted; now left out of the parts list
- R18, R19, R20, R30: LCSC Part # C106232 -> C705627
- R21, R22, R26, R27, R28: LCSC Part # C105872 -> C852856
- R23, R24, R25, R29: LCSC Part # C11702 -> C852624
- R97, R98: LCSC Part # C54920775 -> C100632
Changed lines of the file:
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@@
 			)
 		)
-		(property "LCSC Part #" "C106232"
+		(property "LCSC Part #" "C705627"
 			(at 328.93 210.82 0)
 			(hide yes)
@@
 			)
 		)
-		(property "LCSC Part #" "C11702"
+		(property "LCSC Part #" "C852624"
 			(at 321.31 177.8 90)
 			(hide yes)
@@
 		(on_board yes)
 		(in_pos_files yes)
-		(dnp no)
+		(dnp yes)
 		(fields_autoplaced yes)
 		(property "Reference" "H1"
@@
 			)
 		)
-		(property "LCSC Part #" "C105872"
+		(property "LCSC Part #" "C852856"
 			(at 265.43 46.99 90)
 			(hide yes)
@@
 		(body_style 1)
 		(exclude_from_sim no)
-		(in_bom yes)
+		(in_bom no)
 		(on_board yes)
 		(in_pos_files yes)
-		(dnp no)
+		(dnp yes)
 		(property "Reference" "J4"
 			(at 381 137.16 0)
@@
 			)
 		)
-		(property "LCSC Part #" "C54920775"
+		(property "LCSC Part #" "C100632"
 			(at 217.17 43.18 90)
 			(hide yes)
@@
 			)
 		)
-		(property "LCSC Part #" "C105872"
+		(property "LCSC Part #" "C852856"
 			(at 222.25 36.83 90)
 			(hide yes)
@@
 			)
 		)
-		(property "LCSC Part #" "C105872"
+		(property "LCSC Part #" "C852856"
 			(at 339.09 107.95 0)
 			(hide yes)
@@
 		(body_style 1)
 		(exclude_from_sim no)
-		(in_bom yes)
+		(in_bom no)
 		(on_board yes)
 		(in_pos_files yes)
-		(dnp no)
+		(dnp yes)
 		(property "Reference" "J5"
 			(at 381 196.85 0)
@@
 			)
 		)
-		(property "LCSC Part #" "C54920775"
+		(property "LCSC Part #" "C100632"
 			(at 217.17 48.26 90)
 			(hide yes)
@@
 			)
 		)
-		(property "LCSC Part #" "C106232"
+		(property "LCSC Part #" "C705627"
 			(at 300.99 220.98 0)
 			(hide yes)
@@
 			)
 		)
-		(property "LCSC Part #" "C106232"
+		(property "LCSC Part #" "C705627"
 			(at 328.93 220.98 0)
 			(hide yes)
@@
 			)
 		)
-		(property "LCSC Part #" "C11702"
+		(property "LCSC Part #" "C852624"
 			(at 339.09 127 0)
 			(hide yes)
@@
 			)
 		)
-		(property "LCSC Part #" "C105872"
+		(property "LCSC Part #" "C852856"
 			(at 339.09 116.84 0)
 			(hide yes)
@@
 			)
 		)
-		(property "LCSC Part #" "C105872"
+		(property "LCSC Part #" "C852856"
 			(at 222.25 34.29 90)
 			(hide yes)
@@
 			)
 		)
-		(property "LCSC Part #" "C11702"
+		(property "LCSC Part #" "C852624"
 			(at 321.31 166.37 90)
 			(hide yes)
@@
 		(on_board yes)
 		(in_pos_files yes)
-		(dnp no)
+		(dnp yes)
 		(fields_autoplaced yes)
 		(property "Reference" "H2"
@@
 		(body_style 1)
 		(exclude_from_sim no)
-		(in_bom yes)
+		(in_bom no)
 		(on_board yes)
 		(in_pos_files yes)
-		(dnp no)
+		(dnp yes)
 		(property "Reference" "J2"
 			(at 29.21 271.78 0)
@@
 			)
 		)
-		(property "LCSC Part #" "C106232"
+		(property "LCSC Part #" "C705627"
 			(at 300.99 210.82 0)
 			(hide yes)
@@
 			)
 		)
-		(property "LCSC Part #" "C11702"
+		(property "LCSC Part #" "C852624"
 			(at 321.31 154.94 90)
 			(hide yes)
@@
 		(body_style 1)
 		(exclude_from_sim no)
-		(in_bom yes)
+		(in_bom no)
 		(on_board yes)
 		(in_pos_files yes)
-		(dnp no)
+		(dnp yes)
 		(property "Reference" "J3"
 			(at 255.27 233.68 0)
